Commit message: caught up

File: body.urdf (robot description, URDF)
Before this commit: robot robot, 3 links, 2 joints
Links:
- added link LeftLeg, mass 1; collision box size=1 0.2 0.2; visual box size=1 0.2 0.2
- added link LowBackLeg, mass 1; collision box size=0.2 1 0.2; visual box size=0.2 1 0.2
- added link LowFrontLeg, mass 1; collision box size=0.2 1 0.2; visual box size=0.2 1 0.2
- added link LowLeftLeg, mass 1; collision box size=1 0.2 0.2; visual box size=1 0.2 0.2
- added link LowRightLeg, mass 1; collision box size=1 0.2 0.2; visual box size=1 0.2 0.2
- added link RightLeg, mass 1; collision box size=1 0.2 0.2; visual box size=1 0.2 0.2
- link BackLeg: geometry collision box size=0.2 1 0.2; visual box size=0.2 1 0.2
- link FrontLeg: geometry collision box size=0.2 1 0.2; visual box size=0.2 1 0.2
Joints:
- added joint BackLeg_LowBackLeg: type revolute, parent BackLeg, child LowBackLeg, origin xyz=0 -1 0 rpy=0 0 0, axis 1 0 0, limit lower=-3.14159 upper=3.14159 effort=0.0 velocity=0.0
- added joint FrontLeg_LowFrontLeg: type revolute, parent FrontLeg, child LowFrontLeg, origin xyz=0 1 0 rpy=0 0 0, axis 1 0 0, limit lower=-3.14159 upper=3.14159 effort=0.0 velocity=0.0
- added joint LeftLeg_LowLeftLeg: type revolute, parent LeftLeg, child LowLeftLeg, origin xyz=-1 0 0 rpy=0 0 0, axis 0 1 0, limit lower=-3.14159 upper=3.14159 effort=0.0 velocity=0.0
- added joint RightLeg_LowRightLeg: type revolute, parent RightLeg, child LowRightLeg, origin xyz=1 0 0 rpy=0 0 0, axis 0 1 0, limit lower=-3.14159 upper=3.14159 effort=0.0 velocity=0.0
- added joint Torso_LeftLeg: type revolute, parent Torso, child LeftLeg, origin xyz=-0.5 0 1 rpy=0 0 0, axis 0 1 0, limit lower=-3.14159 upper=3.14159 effort=0.0 velocity=0.0
- added joint Torso_RightLeg: type revolute, parent Torso, child RightLeg, origin xyz=0.5 0 1 rpy=0 0 0, axis 0 1 0, limit lower=-3.14159 upper=3.14159 effort=0.0 velocity=0.0
- joint Torso_BackLeg: axis 0 1 0 -> 1 0 0; origin xyz=-0.5 0 1.0 rpy=0 0 0 -> xyz=0 -0.5 1 rpy=0 0 0
- joint Torso_FrontLeg: axis 0 1 0 -> 1 0 0; origin xyz=0.5 0 1.0 rpy=0 0 0 -> xyz=0 0.5 1 rpy=0 0 0

Commit message: work

File: body.urdf (robot description, URDF)
Before this commit: robot robot, 9 links, 8 joints
Links:
- removed link BackLeg
- removed link FrontLeg
- removed link LeftLeg
- removed link LowBackLeg
- removed link LowFrontLeg
- removed link LowLeftLeg
- removed link LowRightLeg
- removed link RightLeg
- added link Head, mass 1; collision box size=0.6 0.6 0.6; visual box size=0.6 0.6 0.6
- added link LeftBicep, mass 1; collision box size=1 0.25 0.25; visual box size=1 0.25 0.25
- added link LeftCalf, mass 1; collision box size=0.25 0.25 1; visual box size=0.25 0.25 1
- added link LeftForearm, mass 1; collision box size=1 0.25 0.25; visual box size=1 0.25 0.25
- added link LeftHip, mass 1; collision box size=0.25 0.25 0.25; visual box size=0.25 0.25 0.25
- added link LeftShoulder, mass 1; collision box size=0.25 0.25 0.25; visual box size=0.25 0.25 0.25
- added link LeftThigh, mass 1; collision box size=0.25 0.25 1; visual box size=0.25 0.25 1
- added link RightBicep, mass 1; collision box size=1 0.25 0.25; visual box size=1 0.25 0.25
- added link RightCalf, mass 1; collision box size=0.25 0.25 1; visual box size=0.25 0.25 1
- added link RightForearm, mass 1; collision box size=1 0.25 0.25; visual box size=1 0.25 0.25
- added link RightHip, mass 1; collision box size=0.25 0.25 0.25; visual box size=0.25 0.25 0.25
- added link RightShoulder, mass 1; collision box size=0.25 0.25 0.25; visual box size=0.25 0.25 0.25
- added link RightThigh, mass 1; collision box size=0.25 0.25 1; visual box size=0.25 0.25 1
- link Torso: geometry collision box size=1 0.5 2; visual box size=1 0.5 2
Joints:
- removed joint BackLeg_LowBackLeg
- removed joint FrontLeg_LowFrontLeg
- removed joint LeftLeg_LowLeftLeg
- removed joint RightLeg_LowRightLeg
- removed joint Torso_BackLeg
- removed joint Torso_FrontLeg
- removed joint Torso_LeftLeg
- removed joint Torso_RightLeg
- added joint LeftBicep_LeftForearm: type revolute, parent LeftBicep, child LeftForearm, origin xyz=-1 0 0 rpy=0 0 0, axis 0 1 0, limit lower=-3.14159 upper=3.14159 effort=0.0 velocity=0.0
- added joint LeftHip_LeftThigh: type revolute, parent LeftHip, child LeftThigh, origin xyz=0 0 -0.25 rpy=0 0 0, axis 1 0 0, limit lower=-3.14159 upper=3.14159 effort=0.0 velocity=0.0
- added joint LeftShoulder_LeftBicep: type revolute, parent LeftShoulder, child LeftBicep, origin xyz=0 0 0 rpy=0 0 0, axis 0 1 0, limit lower=-3.14159 upper=3.14159 effort=0.0 velocity=0.0
- added joint LeftThigh_LeftCalf: type revolute, parent LeftThigh, child LeftCalf, origin xyz=0 0 -1 rpy=0 0 0, axis 1 0 0, limit lower=-3.14159 upper=3.14159 effort=0.0 velocity=0.0
- added joint RightBicep_RightForearm: type revolute, parent RightBicep, child RightForearm, origin xyz=1 0 0 rpy=0 0 0, axis 0 1 0, limit lower=-3.14159 upper=3.14159 effort=0.0 velocity=0.0
- added joint RightHip_RightThigh: type revolute, parent RightHip, child RightThigh, origin xyz=0 0 -0.25 rpy=0 0 0, axis 1 0 0, limit lower=-3.14159 upper=3.14159 effort=0.0 velocity=0.0
- added joint RightShoulder_RightBicep: type revolute, parent RightShoulder, child RightBicep, origin xyz=0 0 0 rpy=0 0 0, axis 0 1 0, limit lower=-3.14159 upper=3.14159 effort=0.0 velocity=0.0
- added joint RightThigh_RightCalf: type revolute, parent RightThigh, child RightCalf, origin xyz=0 0 -1 rpy=0 0 0, axis 1 0 0, limit lower=-3.14159 upper=3.14159 effort=0.0 velocity=0.0
- added joint Torso_Head: type revolute, parent Torso, child Head, origin xyz=0 0 4.5 rpy=0 0 0, axis 1 0 0, limit lower=-3.14159 upper=3.14159 effort=0.0 velocity=0.0
- added joint Torso_LeftHip: type revolute, parent Torso, child LeftHip, origin xyz=0.4 0 2.5 rpy=0 0 0, axis 0 1 0, limit lower=-3.14159 upper=3.14159 effort=0.0 velocity=0.0
- added joint Torso_LeftShoulder: type revolute, parent Torso, child LeftShoulder, origin xyz=-0.5 0 4.5 rpy=0 0 0, axis 0 0 1, limit lower=-3.14159 upper=3.14159 effort=0.0 velocity=0.0
- added joint Torso_RightHip: type revolute, parent Torso, child RightHip, origin xyz=-0.4 0 2.5 rpy=0 0 0, axis 0 1 0, limit lower=-3.14159 upper=3.14159 effort=0.0 velocity=0.0
- added joint Torso_RightShoulder: type revolute, parent Torso, child RightShoulder, origin xyz=0.5 0 4.5 rpy=0 0 0, axis 0 0 1, limit lower=-3.14159 upper=3.14159 effort=0.0 velocity=0.0
